Commit message: modifications

File: xarm_description/urdf/gripper/xarm_gripper.urdf.xacro (robot description, xacro)
@@ -1,5 +1,5 @@
 <?xml version="1.0"?>
 <robot xmlns:xacro="http://ros.org/wiki/xacro" name="xarm_gripper">
-  <xacro:macro name="xarm_gripper_urdf" params="prefix:='' attach_to:='' attach_xyz:='0 0 0' attach_rpy:='0 0 0' ">
+  <xacro:macro name="xarm_gripper_urdf" params="prefix:='' attach_to:='link_eef' attach_xyz:='0 0 0' attach_rpy:='0 0 0' ">
     <xacro:unless value="${attach_to == ''}">
       <joint name="${prefix}gripper_fix" type="fixed">
@@ -184,5 +184,5 @@
     <link name="${prefix}link_tcp" />
     <joint name="${prefix}joint_tcp" type="fixed">
-      <origin xyz="0 0 0.172" rpy="0 0 0" />
+      <origin xyz="0 0 0.12" rpy="0 0 0" />
       <parent link="${prefix}xarm_gripper_base_link" />
       <child link="${prefix}link_tcp" />

File: xarm_description/urdf/xarm_device.urdf.xacro (robot description, xacro)
@@ -20,5 +20,5 @@
   <xacro:arg name="add_d435i_links" default="true"/>
   <xacro:arg name="use_gazebo_camera" default="false"/>
-  <xacro:arg name="add_other_geometry" default="false"/>
+  <xacro:arg name="add_other_geometry" default="True"/>
   <xacro:arg name="geometry_type" default="box"/>
   <xacro:arg name="geometry_mass" default="0.1"/>

File: xarm_description/urdf/xarm_device_macro.xacro (robot description, xacro)
@@ -67,10 +67,232 @@
     <xacro:if value="${attach_to == 'world' and create_attach_link}">
       <link name="world" />
-    </xacro:if>
-    <joint name="${prefix}world_joint" type="fixed">
-      <parent link="${attach_to}" />
-      <child link="${prefix}link_base" />
-      <origin xyz="${attach_xyz}" rpy="${attach_rpy}" />
-    </joint>
+      <link name="${prefix}base" />
+      <joint name="${prefix}world_joint" type="fixed">
+        <parent link="${attach_to}" />
+        <child link="${prefix}base" />
+        <origin xyz="0 0 0" rpy="0 0 0" />
+      </joint>
+    </xacro:if>
+    <link name="${prefix}base_cylinder">
+      <visual>
+        <geometry>
+          <cylinder radius="0.07" length="1"/>
+        </geometry>
+        <origin xyz="0 0 -0.5" rpy="0 0 0"/>
+      </visual>
+      <collision>
+        <geometry>
+          <cylinder radius="0.07" length="1"/>
+        </geometry>
+        <origin xyz="0 0 -0.5" rpy="0 0 0"/>
+      </collision>
+    </link>
+<link name="${prefix}table1">
+  <visual>
+    <geometry>
+      <box size="0.5 0.3 0.05"/>
+    </geometry>
+  </visual>
+  <collision>
+    <geometry>
+      <box size="0.5 0.3 0.05"/>
+    </geometry>
+  </collision>
+  <inertial>
+    <mass value="5.0"/>
+    <origin xyz="0 0 0"/>
+    <inertia ixx="0.1" ixy="0.0" ixz="0.0"
+             iyy="0.1" iyz="0.0"
+             izz="0.1"/>
+  </inertial>
+</link>
+<joint name="${prefix}world_table" type="fixed">
+    <parent link="world"/>
+    <child link="${prefix}table1"/>
+    <origin xyz="0.75 0 0.75" rpy="0 0 0"/>
+</joint>
+<!-- Table Legs -->
+<link name="${prefix}leg_1">
+  <visual>
+    <geometry>
+      <cylinder radius="0.025" length="0.7"/>
+    </geometry>
+  </visual>
+  <collision>
+    <geometry>
+      <cylinder radius="0.025" length="0.7"/>
+    </geometry>
+  </collision>
+</link>
+<link name="${prefix}leg_2">
+  <visual>
+    <geometry>
+      <cylinder radius="0.025" length="0.7"/>
+    </geometry>
+  </visual>
+  <collision>
+    <geometry>
+      <cylinder radius="0.025" length="0.7"/>
+    </geometry>
+  </collision>
+</link>
+<link name="${prefix}leg_3">
+  <visual>
+    <geometry>
+      <cylinder radius="0.025" length="0.7"/>
+    </geometry>
+  </visual>
+  <collision>
+    <geometry>
+      <cylinder radius="0.025" length="0.7"/>
+    </geometry>
+  </collision>
+</link>
+<link name="${prefix}leg_4">
+  <visual>
+    <geometry>
+      <cylinder radius="0.025" length="0.7"/>
+    </geometry>
+  </visual>
+  <collision>
+    <geometry>
+      <cylinder radius="0.025" length="0.7"/>
+    </geometry>
+  </collision>
+</link>
+<!-- Fixed Joints for Legs -->
+<joint name="${prefix}table_leg_1" type="fixed">
+  <parent link="${prefix}table1"/>
+  <child link="${prefix}leg_1"/>
+  <origin xyz="0.225 0.125 -0.375" rpy="0 0 0"/>
+</joint>
+<joint name="${prefix}table_leg_2" type="fixed">
+  <parent link="${prefix}table1"/>
+  <child link="${prefix}leg_2"/>
+  <origin xyz="-0.225 0.125 -0.375" rpy="0 0 0"/>
+</joint>
+<joint name="${prefix}table_leg_3" type="fixed">
+  <parent link="${prefix}table1"/>
+  <child link="${prefix}leg_3"/>
+  <origin xyz="0.225 -0.125 -0.375" rpy="0 0 0"/>
+</joint>
+<joint name="${prefix}table_leg_4" type="fixed">
+  <parent link="${prefix}table1"/>
+  <child link="${prefix}leg_4"/>
+  <origin xyz="-0.225 -0.125 -0.375" rpy="0 0 0"/>
+</joint>
+<joint name="${prefix}link_base_to_cylinder" type="fixed">
+  <parent link="${prefix}base"/>
+  <child link="${prefix}base_cylinder"/>
+  <origin xyz="0 0 1" rpy="0 0 0"/>
+</joint>
+<joint name="${prefix}cylinder_link" type="fixed">
+  <parent link="${prefix}base_cylinder" />
+  <child link="${prefix}link_base" />
+  <origin xyz="0 0 0" rpy="0 0 0" />
+</joint>
+<!-- Second Table Top -->
+<link name="${prefix}table_2">
+  <visual>
+    <geometry>
+      <box size="0.5 0.3 0.05"/>
+    </geometry>
+  </visual>
+  <collision>
+    <geometry>
+      <box size="0.5 0.3 0.05"/>
+    </geometry>
+  </collision>
+  <inertial>
+    <mass value="5.0"/>
+    <origin xyz="0 0 0"/>
+    <inertia ixx="0.1" ixy="0.0" ixz="0.0"
+             iyy="0.1" iyz="0.0"
+             izz="0.1"/>
+  </inertial>
+</link>
+<!-- Fixed Joint to World -->
+<joint name="${prefix}world_table_2" type="fixed">
+  <parent link="world"/>
+  <child link="${prefix}table_2"/>
+  <origin xyz="0.75 0.5 0.75" rpy="0 0 0"/>
+</joint>
+<!-- Second Table Legs -->
+<link name="${prefix}leg_21">
+  <visual>
+    <geometry>
+      <cylinder radius="0.025" length="0.70"/>
+    </geometry>
+  </visual>
+  <collision>
+    <geometry>
+      <cylinder radius="0.025" length="0.70"/>
+    </geometry>
+  </collision>
+</link>
+<joint name="${prefix}leg_1_joint" type="fixed">
+  <parent link="${prefix}table_2"/>
+  <child link="${prefix}leg_21"/>
+  <origin xyz="0.2 0.075 -0.375"/>
+</joint>
+<link name="${prefix}leg_22">
+  <visual>
+    <geometry>
+      <cylinder radius="0.025" length="0.70"/>
+    </geometry>
+  </visual>
+  <collision>
+    <geometry>
+      <cylinder radius="0.025" length="0.70"/>
+    </geometry>
+  </collision>
+</link>
+<joint name="${prefix}leg_2_joint" type="fixed">
+  <parent link="${prefix}table_2"/>
+  <child link="${prefix}leg_22"/>
+  <origin xyz="-0.2 0.075 -0.375"/>
+</joint>
+<link name="${prefix}leg_23">
+  <visual>
+    <geometry>
+      <cylinder radius="0.025" length="0.70"/>
+    </geometry>
+  </visual>
+  <collision>
+    <geometry>
+      <cylinder radius="0.025" length="0.70"/>
+    </geometry>
+  </collision>
+</link>
+<joint name="${prefix}leg_3_joint" type="fixed">
+  <parent link="${prefix}table_2"/>
+  <child link="${prefix}leg_23"/>
+  <origin xyz="0.2 -0.075 -0.375"/>
+</joint>
+<link name="${prefix}leg_24">
+  <visual>
+    <geometry>
+      <cylinder radius="0.025" length="0.70"/>
+    </geometry>
+  </visual>
+  <collision>
+    <geometry>
+      <cylinder radius="0.025" length="0.70"/>
+    </geometry>
+  </collision>
+</link>
+<joint name="${prefix}leg_4_joint" type="fixed">
+  <parent link="${prefix}table_2"/>
+  <child link="${prefix}leg_24"/>
+  <origin xyz="-0.2 -0.075 -0.375"/>
+</joint>
+<gazebo reference="table1">
+    <static>true</static>  <!-- Ensures it doesn’t move -->
+    <material>Gazebo/Wood</material>
+</gazebo>
+<gazebo reference="table_2">
+    <static>true</static>  <!-- Ensures it doesn’t move -->
+    <material>Gazebo/Wood</material>
+</gazebo>
     <xacro:if value="${effort_control}">
       <xacro:property name="hard_interface" value="EffortJointInterface" />

File: xarm_moveit_config/srdf/_xarm6_macro.srdf.xacro (robot description, xacro)
@@ -93,4 +93,9 @@
       <disable_collisions link1="${prefix}left_finger" link2="${prefix}xarm_gripper_base_link" reason="Never" />
       <disable_collisions link1="${prefix}left_inner_knuckle" link2="${prefix}left_outer_knuckle" reason="Never" />
+      <disable_collisions link1="grip" link2="link_tcp" reason="Never" />
+      <disable_collisions link1="${prefix}table1" link2="${prefix}leg_1" reason="adjacent fixed joint"/>
+      <disable_collisions link1="${prefix}table1" link2="${prefix}leg_2" reason="adjacent fixed joint"/>
+      <disable_collisions link1="${prefix}table1" link2="${prefix}leg_3" reason="adjacent fixed joint"/>
+      <disable_collisions link1="${prefix}table1" link2="${prefix}leg_4" reason="adjacent fixed joint"/>
       <disable_collisions link1="${prefix}left_inner_knuckle" link2="${prefix}link4" reason="Never" />
       <disable_collisions link1="${prefix}left_inner_knuckle" link2="${prefix}link5" reason="Never" />
@@ -106,4 +111,9 @@
       <disable_collisions link1="${prefix}left_outer_knuckle" link2="${prefix}right_outer_knuckle" reason="Never" />
       <disable_collisions link1="${prefix}left_outer_knuckle" link2="${prefix}xarm_gripper_base_link" reason="Adjacent" />
+      <disable_collisions link1="base_cylinder" link2="link_base" reason="adjacent fixed joint"/>
+      <disable_collisions link1="table_2" link2="leg_21" reason="adjacent fixed joint"/>
+      <disable_collisions link1="table_2" link2="leg_22" reason="adjacent fixed joint"/>
+      <disable_collisions link1="table_2" link2="leg_23" reason="adjacent fixed joint"/>
+      <disable_collisions link1="table_2" link2="leg_24" reason="adjacent fixed joint"/>
       <disable_collisions link1="${prefix}link4" link2="${prefix}right_finger" reason="Never" />
       <disable_collisions link1="${prefix}link4" link2="${prefix}right_inner_knuckle" reason="Never" />
@@ -123,4 +133,5 @@
       <disable_collisions link1="${prefix}right_inner_knuckle" link2="${prefix}xarm_gripper_base_link" reason="Adjacent" />
       <disable_collisions link1="${prefix}right_outer_knuckle" link2="${prefix}xarm_gripper_base_link" reason="Adjacent" />
+      <disable_collisions link1="${prefix}link_eef" link2="${prefix}link6" reason="Never" />
       <disable_collisions link1="${prefix}link_eef" link2="${prefix}left_finger" reason="Never" />
       <disable_collisions link1="${prefix}link_eef" link2="${prefix}left_inner_knuckle" reason="Never" />
